Commit message: added turtlebot3_msgs and DynamixelSDK as submodules instead

File: turtlebot3_description/urdf/tb3_conveyor_macro.xacro (robot description, xacro)
@@ -33,5 +33,5 @@
     <color rgba="1.0 1.0 1.0 1.0"/>
   </material>
-  <!-- <xacro:macro name="wheel" params="name xyz rpy">
+  <xacro:macro name="wheel" params="name xyz rpy">
     <link name="wheel_${name}_link">
       <visual>
@@ -60,5 +60,5 @@
       <axis xyz="0 0 1"/>
     </joint>
-  </xacro:macro> -->
+  </xacro:macro>
   <xacro:macro name="swerve_wheel" params="name xy yaw">
     <link name = "pivot_${name}_link"/>

File: turtlebot3_description/urdf/turtlebot3_conveyor.urdf.xacro (robot description, xacro)
@@ -30,6 +30,6 @@
     </inertial>
   </link>
-  <!-- <xacro:wheel name="left" xyz="0.0 0.08 0.023" rpy="-1.57 0 0"/> -->
-  <!-- <xacro:wheel name="right" xyz="0.0 -0.08 0.023" rpy="-1.57 0 0"/> -->
+  <xacro:wheel name="left" xyz="0.0 0.08 0.023" rpy="-1.57 0 0"/>
+  <xacro:wheel name="right" xyz="0.0 -0.08 0.023" rpy="-1.57 0 0"/>
   <xacro:swerve_wheel name="right_front" xy="${base_length/2} ${-base_length/2}" yaw="0.707"/>
   <xacro:swerve_wheel name="left_front" xy="${base_length/2} ${base_length/2}" yaw="${0.707+1.57}"/>

Commit message: publishes joints onto rviz2 and can now be used for odom programming

File: turtlebot3_description/urdf/tb3_conveyor_macro.xacro (robot description, xacro)
@@ -33,5 +33,5 @@
     <color rgba="1.0 1.0 1.0 1.0"/>
   </material>
-  <xacro:macro name="wheel" params="name xyz rpy">
+  <!-- <xacro:macro name="wheel" params="name xyz rpy">
     <link name="wheel_${name}_link">
       <visual>
@@ -60,5 +60,5 @@
       <axis xyz="0 0 1"/>
     </joint>
-  </xacro:macro>
+  </xacro:macro> -->
   <xacro:macro name="swerve_wheel" params="name xy yaw">
     <link name = "pivot_${name}_link"/>
@@ -93,5 +93,5 @@
       <parent link="pivot_${name}_link"/>
       <child link="wheel_${name}_link"/>
-      <origin xyz="0 0 0" rpy="-1.57 0 0"/>
+      <origin xyz="0 0 0" rpy="-1.57 0 3.14"/>
       <axis xyz="0 0 1"/>
     </joint>

File: turtlebot3_description/urdf/turtlebot3_conveyor.urdf.xacro (robot description, xacro)
@@ -30,10 +30,10 @@
     </inertial>
   </link>
-  <xacro:wheel name="left" xyz="0.0 0.08 0.023" rpy="-1.57 0 0"/>
-  <xacro:wheel name="right" xyz="0.0 -0.08 0.023" rpy="-1.57 0 0"/>
-  <xacro:swerve_wheel name="right_front" xy="${base_length/2} ${-base_length/2}" yaw="0.707"/>
-  <xacro:swerve_wheel name="left_front" xy="${base_length/2} ${base_length/2}" yaw="${0.707+1.57}"/>
-  <xacro:swerve_wheel name="left_rear" xy="${-base_length/2} ${base_length/2}" yaw="${0.707+1.57*2}"/>
-  <xacro:swerve_wheel name="right_rear" xy="${-base_length/2} ${-base_length/2}" yaw="${0.707+1.57*3}"/>
+  <!-- <xacro:wheel name="left" xyz="0.0 0.08 0.023" rpy="-1.57 0 0"/>
+  <xacro:wheel name="right" xyz="0.0 -0.08 0.023" rpy="-1.57 0 0"/> -->
+  <xacro:swerve_wheel name="right_front" xy="${base_length/2} ${-base_length/2}" yaw="0.785"/>
+  <xacro:swerve_wheel name="left_front" xy="${base_length/2} ${base_length/2}" yaw="${0.785+1.571}"/>
+  <xacro:swerve_wheel name="left_rear" xy="${-base_length/2} ${base_length/2}" yaw="${0.785+1.571*2}"/>
+  <xacro:swerve_wheel name="right_rear" xy="${-base_length/2} ${-base_length/2}" yaw="${0.785+1.571*3}"/>
   <joint name="imu_joint" type="fixed">
     <parent link="base_link"/>
