Commit message: yayy kinda worksss

File: turtlebot3_description/urdf/turtlebot3_conveyor.urdf.xacro (robot description, xacro)
@@ -8,5 +8,5 @@
     <parent link="base_footprint"/>
     <child link="base_link"/>
-    <origin xyz="0.0 0.0 0.010" rpy="0 0 0"/>
+    <origin xyz="0.87 0.0 0.010" rpy="0 0 0"/>
   </joint>
   <link name="base_link">
@@ -45,5 +45,5 @@
     <parent link="base_link"/>
     <child link="base_scan"/>
-    <origin xyz="0 0 0.10" rpy="0 0 0"/>
+    <origin xyz="0.09 0 0" rpy="0 0 3.14"/>
   </joint>
   <link name="base_scan">

Commit message: updated odom base frame in conveyor.yaml to base_link instead of base footprint

File: turtlebot3_description/urdf/turtlebot3_conveyor.urdf.xacro (robot description, xacro)
@@ -6,7 +6,7 @@
   <link name="base_footprint"/>
   <joint name="base_joint" type="fixed">
-    <parent link="base_footprint"/>
-    <child link="base_link"/>
-    <origin xyz="0.87 0.0 0.010" rpy="0 0 0"/>
+    <parent link="base_link"/>
+    <child link="base_footprint"/>
+    <origin xyz="-0.87 0.0 0.010" rpy="0 0 0"/>
   </joint>
   <link name="base_link">

Commit message: first commit for this branch. transforms are different for base_footprint

File: turtlebot3_description/urdf/turtlebot3_conveyor.urdf.xacro (robot description, xacro)
@@ -8,5 +8,5 @@
     <parent link="base_link"/>
     <child link="base_footprint"/>
-    <origin xyz="-0.87 0.0 0.010" rpy="0 0 0"/>
+    <origin xyz="0.0 0.0 0.010" rpy="0 0 0"/>
   </joint>
   <link name="base_link">

Commit message: re added base footprint offset

File: turtlebot3_description/urdf/turtlebot3_conveyor.urdf.xacro (robot description, xacro)
@@ -8,5 +8,5 @@
     <parent link="base_link"/>
     <child link="base_footprint"/>
-    <origin xyz="0.0 0.0 0.010" rpy="0 0 0"/>
+    <origin xyz="-0.87 0.0 0.010" rpy="0 0 0"/>
   </joint>
   <link name="base_link">

Commit message: adjusted depth cam angle in urdf

File: turtlebot3_description/urdf/turtlebot3_conveyor.urdf.xacro (robot description, xacro)
@@ -42,4 +42,10 @@
   </joint>
   <link name="imu_link"/>
+  <joint name="camera_joint" type="fixed">
+    <parent link="base_link"/>
+    <child link="camera_link"/>
+    <origin xyz="0.03 0 0.2" rpy="0 -0.349 0"/>
+  </joint>
+  <link name="camera_link"/>
   <joint name="scan_joint" type="fixed">
     <parent link="base_link"/>

Commit message: changed base_footprint to be main parent

File: turtlebot3_description/urdf/turtlebot3_conveyor.urdf.xacro (robot description, xacro)
@@ -6,6 +6,6 @@
   <link name="base_footprint"/>
   <joint name="base_joint" type="fixed">
-    <parent link="base_link"/>
-    <child link="base_footprint"/>
+    <parent link="base_footprint"/>
+    <child link="base_link"/>
     <origin xyz="0.0 0.0 0.010" rpy="0 0 0"/>
   </joint>
@@ -42,4 +42,10 @@
   </joint>
   <link name="imu_link"/>
+  <joint name="camera_joint" type="fixed">
+    <parent link="base_link"/>
+    <child link="camera_link"/>
+    <origin xyz="0.03 0 0.2" rpy="0 -0.349 0"/>
+  </joint>
+  <link name="camera_link"/>
   <joint name="scan_joint" type="fixed">
     <parent link="base_link"/>

Commit message: changed frames for better costmap

File: turtlebot3_description/urdf/turtlebot3_conveyor.urdf.xacro (robot description, xacro)
@@ -4,9 +4,16 @@
   <!-- <xacro:include filename="$(find turtlebot3_description)/urdf/common_properties.urdf"/> -->
   <xacro:include filename="tb3_conveyor_macro.xacro"/>
+  <xacro:property name="basefp_to_baselink" value="0.87"/>
+  <link name="robo_base"/>
+  <joint name="robo_joint" type="fixed">
+    <parent link="robo_base"/>
+    <child link="base_footprint"/>
+    <origin xyz="-${basefp_to_baselink} 0.0 0.0" rpy="0 0 0"/>
+  </joint>
   <link name="base_footprint"/>
   <joint name="base_joint" type="fixed">
-    <parent link="base_link"/>
-    <child link="base_footprint"/>
-    <origin xyz="-0.87 0.0 0.010" rpy="0 0 0"/>
+    <parent link="base_footprint"/>
+    <child link="base_link"/>
+    <origin xyz="${basefp_to_baselink} 0.0 0.010" rpy="0 0 0"/>
   </joint>
   <link name="base_link">
